File: RamanCCDBoard/RamanCCDBoard.kicad_pcb (KiCad board)
At the start: 2 copper layers, 61 x 15.2 mm, 10 parts, among them J1 Conn_01x03_Pin, Q2 KSA1015YTA, U1 ILX511

Commit message: board review changes
Changed lines of the file:
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@@
   (via (at 80.01 24.638) (size 0.8) (drill 0.4) (layers "F.Cu" "B.Cu") (net 2))
   (segment (start 83.365 24.638) (end 80.01 24.638) (width 0.254) (layer "B.Cu") (net 2))
-  (segment (start 53.848 23.782) (end 53.848 23.876) (width 0.25) (layer "B.Cu") (net 3))
+  (segment (start 77.056 25.654) (end 77.216 25.654) (width 0.25) (layer "B.Cu") (net 3))
+  (segment (start 57.404 23.782) (end 57.404 23.876) (width 0.25) (layer "B.Cu") (net 3))
   (segment (start 58.674 23.876) (end 58.928 23.876) (width 0.254) (layer "B.Cu") (net 3))
-  (segment (start 55.626 22.004) (end 53.848 23.782) (width 0.25) (layer "B.Cu") (net 3))
   (segment (start 80.772 27.94) (end 80.772 28.956) (width 0.254) (layer "B.Cu") (net 3))
-  (segment (start 56.388 23.782) (end 56.388 23.876) (width 0.25) (layer "B.Cu") (net 3))
+  (segment (start 60.706 22.004) (end 62.484 23.782) (width 0.25) (layer "B.Cu") (net 3))
+  (segment (start 58.166 22.004) (end 59.944 23.782) (width 0.25) (layer "B.Cu") (net 3))
+  (segment (start 62.484 23.782) (end 62.484 23.876) (width 0.25) (layer "B.Cu") (net 3))
   (segment (start 80.264 25.654) (end 80.772 26.162) (width 0.254) (layer "B.Cu") (net 3))
   (segment (start 75.946 32.004) (end 77.47 30.48) (width 0.254) (layer "B.Cu") (net 3))
@@
   (segment (start 80.264 25.654) (end 82.095 25.654) (width 0.254) (layer "B.Cu") (net 3))
   (segment (start 77.47 30.48) (end 69.85 30.48) (width 0.254) (layer "B.Cu") (net 3))
-  (segment (start 59.436 26.416) (end 56.896 23.876) (width 0.25) (layer "B.Cu") (net 3))
   (segment (start 52.9825 23.876) (end 53.848 23.876) (width 0.25) (layer "B.Cu") (net 3))
-  (segment (start 73.406 22.004) (end 69.756 25.654) (width 0.254) (layer "B.Cu") (net 3))
-  (segment (start 60.706 22.004) (end 58.928 23.782) (width 0.25) (layer "B.Cu") (net 3))
+  (segment (start 61.976 23.876) (end 62.484 23.876) (width 0.254) (layer "B.Cu") (net 3))
   (segment (start 79.248 30.48) (end 77.47 30.48) (width 0.254) (layer "B.Cu") (net 3))
-  (segment (start 58.166 22.004) (end 56.388 23.782) (width 0.25) (layer "B.Cu") (net 3))
+  (segment (start 62.484 23.876) (end 66.548 23.876) (width 0.254) (layer "B.Cu") (net 3))
+  (segment (start 77.216 25.654) (end 80.264 25.654) (width 0.254) (layer "B.Cu") (net 3))
   (segment (start 56.896 23.876) (end 56.388 23.876) (width 0.254) (layer "B.Cu") (net 3))
   (segment (start 57.404 23.876) (end 58.674 23.876) (width 0.254) (layer "B.Cu") (net 3))
@@
   (segment (start 80.772 26.162) (end 80.772 27.94) (width 0.254) (layer "B.Cu") (net 3))
   (segment (start 82.095 25.654) (end 83.365 26.924) (width 0.254) (layer "B.Cu") (net 3))
+  (segment (start 59.944 23.876) (end 61.976 23.876) (width 0.254) (layer "B.Cu") (net 3))
   (segment (start 80.772 28.956) (end 79.248 30.48) (width 0.254) (layer "B.Cu") (net 3))
-  (segment (start 58.928 23.782) (end 58.928 23.876) (width 0.25) (layer "B.Cu") (net 3))
+  (segment (start 59.436 26.416) (end 61.976 23.876) (width 0.25) (layer "B.Cu") (net 3))
+  (segment (start 59.944 23.782) (end 59.944 23.876) (width 0.25) (layer "B.Cu") (net 3))
   (segment (start 82.042 29.21) (end 83.365 29.21) (width 0.254) (layer "B.Cu") (net 3))
   (segment (start 68.326 25.654) (end 71.628 25.654) (width 0.254) (layer "B.Cu") (net 3))
+  (segment (start 73.406 22.004) (end 77.056 25.654) (width 0.25) (layer "B.Cu") (net 3))
   (segment (start 69.756 25.654) (end 72.136 25.654) (width 0.254) (layer "B.Cu") (net 3))
   (segment (start 57.404 23.876) (end 56.896 23.876) (width 0.254) (layer "B.Cu") (net 3))
   (segment (start 80.772 27.94) (end 82.042 29.21) (width 0.254) (layer "B.Cu") (net 3))
   (segment (start 58.928 23.876) (end 59.944 23.876) (width 0.254) (layer "B.Cu") (net 3))
+  (segment (start 72.136 25.654) (end 77.216 25.654) (width 0.254) (layer "B.Cu") (net 3))
   (segment (start 66.548 23.876) (end 68.326 25.654) (width 0.254) (layer "B.Cu") (net 3))
   (segment (start 69.85 30.48) (end 68.326 32.004) (width 0.254) (layer "B.Cu") (net 3))
-  (segment (start 59.944 23.876) (end 66.548 23.876) (width 0.254) (layer "B.Cu") (net 3))
-  (segment (start 72.136 25.654) (end 80.264 25.654) (width 0.254) (layer "B.Cu") (net 3))
   (segment (start 71.628 25.654) (end 72.136 25.654) (width 0.254) (layer "B.Cu") (net 3))
+  (segment (start 55.626 22.004) (end 57.404 23.782) (width 0.25) (layer "B.Cu") (net 3))
   (segment (start 65.024 30.226) (end 63.246 32.004) (width 0.254) (layer "F.Cu") (net 4))
   (via (at 65.024 30.226) (size 0.8) (drill 0.4) (layers "F.Cu" "B.Cu") (net 4))

Commit message: generated gerbs
Routing:
- net +5V: track 75.8 -> 78.3 mm
Changed lines of the file:
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@@
   (gr_arc (start 98.805999 30.733999) (mid 97.690076 33.428076) (end 94.995999 34.543999)
     (stroke (width 0.2) (type default)) (layer "Edge.Cuts"))
-  (gr_text "CCD Breakout, Rev2\nMars Rover Design Team\nMissouri S&T, 2024\nCaleb Ehlers" (at 89.916 26.924 90) (layer "B.SilkS")
-    (effects (font (size 0.635 0.635) (thickness 0.127) bold) (justify bottom mirror))
+  (gr_text "CCD Breakout, Rev2\nMars Rover Design Team\nMissouri S&T, 2024\nCaleb Ehlers" (at 89.662 21.082 90) (layer "B.SilkS")
+    (effects (font (size 0.635 0.635) (thickness 0.127) bold) (justify left bottom mirror))
   )
   (gr_text "gnd" (at 79.248 29.718) (layer "B.SilkS")
@@
   (segment (start 60.706 22.004) (end 62.484 23.782) (width 0.25) (layer "B.Cu") (net 3))
   (segment (start 58.166 22.004) (end 59.944 23.782) (width 0.25) (layer "B.Cu") (net 3))
+  (segment (start 73.406 27.432) (end 75.184 25.654) (width 0.254) (layer "B.Cu") (net 3))
   (segment (start 62.484 23.782) (end 62.484 23.876) (width 0.25) (layer "B.Cu") (net 3))
   (segment (start 80.264 25.654) (end 80.772 26.162) (width 0.254) (layer "B.Cu") (net 3))
@@
   (segment (start 82.095 25.654) (end 83.365 26.924) (width 0.254) (layer "B.Cu") (net 3))
   (segment (start 59.944 23.876) (end 61.976 23.876) (width 0.254) (layer "B.Cu") (net 3))
+  (segment (start 75.184 25.654) (end 77.216 25.654) (width 0.254) (layer "B.Cu") (net 3))
   (segment (start 80.772 28.956) (end 79.248 30.48) (width 0.254) (layer "B.Cu") (net 3))
   (segment (start 59.436 26.416) (end 61.976 23.876) (width 0.25) (layer "B.Cu") (net 3))
@@
   (segment (start 80.772 27.94) (end 82.042 29.21) (width 0.254) (layer "B.Cu") (net 3))
   (segment (start 58.928 23.876) (end 59.944 23.876) (width 0.254) (layer "B.Cu") (net 3))
-  (segment (start 72.136 25.654) (end 77.216 25.654) (width 0.254) (layer "B.Cu") (net 3))
   (segment (start 66.548 23.876) (end 68.326 25.654) (width 0.254) (layer "B.Cu") (net 3))
   (segment (start 69.85 30.48) (end 68.326 32.004) (width 0.254) (layer "B.Cu") (net 3))
+  (segment (start 72.136 25.654) (end 75.184 25.654) (width 0.254) (layer "B.Cu") (net 3))
   (segment (start 71.628 25.654) (end 72.136 25.654) (width 0.254) (layer "B.Cu") (net 3))
   (segment (start 55.626 22.004) (end 57.404 23.782) (width 0.25) (layer "B.Cu") (net 3))
